File: Indication.kicad_sch (KiCad schematic)
At the start: 12 parts, among them Q4 AO3400A

Commit message: feat: finish schematic (Full)
Parts:
- BZ1: footprint Buzzer_Beeper:Buzzer_CUI_CMT-8504-SMT-TR -> Buzzer_Beeper:Buzzer_CUI_CPT-9019S-SMT
- D15: renamed from D14; value LED -> LED_RED
- D16: renamed from D15; value LED -> LED_GREEN
- renumbered D16 to D14, Q4 to Q5, R38 to R33, R37 to R34, R36 to R35, R35 to R36, R39 to R37, R33 to R38, R34 to R39
Changed lines of the file:
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@@
 		(dnp no)
 		(fields_autoplaced yes)
-		(property "Reference" "R34"
+		(property "Reference" "R39"
 			(at 109.22 68.58 0)
 			(show_name no)
@@
 			(project "UNSW_Rocketry_Senior_Flight_Computer"
 				(path "/9e0253f5-fba5-4205-8256-7fc47a91dd1e/57914cc3-efa9-43f1-a4d3-11a42d51adab"
-					(reference "R34")
+					(reference "R39")
 					(unit 1)
 				)
@@
 		(dnp no)
 		(fields_autoplaced yes)
-		(property "Reference" "#PWR088"
+		(property "Reference" "#PWR092"
 			(at 133.35 74.93 0)
 			(hide yes)
@@
 			(project "UNSW_Rocketry_Senior_Flight_Computer"
 				(path "/9e0253f5-fba5-4205-8256-7fc47a91dd1e/57914cc3-efa9-43f1-a4d3-11a42d51adab"
-					(reference "#PWR088")
+					(reference "#PWR092")
 					(unit 1)
 				)
@@
 		(dnp no)
 		(fields_autoplaced yes)
-		(property "Reference" "#PWR090"
+		(property "Reference" "#PWR089"
 			(at 132.08 99.06 0)
 			(hide yes)
@@
 			(project "UNSW_Rocketry_Senior_Flight_Computer"
 				(path "/9e0253f5-fba5-4205-8256-7fc47a91dd1e/57914cc3-efa9-43f1-a4d3-11a42d51adab"
-					(reference "#PWR090")
+					(reference "#PWR089")
 					(unit 1)
 				)
@@
 		(dnp no)
 		(fields_autoplaced yes)
-		(property "Reference" "Q4"
+		(property "Reference" "Q5"
 			(at 114.3 142.24 90)
 			(show_name no)
@@
 			(project "UNSW_Rocketry_Senior_Flight_Computer"
 				(path "/9e0253f5-fba5-4205-8256-7fc47a91dd1e/57914cc3-efa9-43f1-a4d3-11a42d51adab"
-					(reference "Q4")
+					(reference "Q5")
 					(unit 1)
 				)
@@
 		(dnp no)
 		(fields_autoplaced yes)
-		(property "Reference" "#PWR091"
+		(property "Reference" "#PWR090"
 			(at 132.08 104.14 0)
 			(hide yes)
@@
 			(project "UNSW_Rocketry_Senior_Flight_Computer"
 				(path "/9e0253f5-fba5-4205-8256-7fc47a91dd1e/57914cc3-efa9-43f1-a4d3-11a42d51adab"
-					(reference "#PWR091")
+					(reference "#PWR090")
 					(unit 1)
 				)
@@
 		(dnp no)
 		(fields_autoplaced yes)
-		(property "Reference" "#PWR087"
+		(property "Reference" "#PWR091"
 			(at 133.35 55.88 0)
 			(hide yes)
@@
 			(project "UNSW_Rocketry_Senior_Flight_Computer"
 				(path "/9e0253f5-fba5-4205-8256-7fc47a91dd1e/57914cc3-efa9-43f1-a4d3-11a42d51adab"
-					(reference "#PWR087")
+					(reference "#PWR091")
 					(unit 1)
 				)
@@
 		(dnp no)
 		(fields_autoplaced yes)
-		(property "Reference" "#PWR093"
+		(property "Reference" "#PWR087"
 			(at 97.79 138.43 0)
 			(hide yes)
@@
 			(project "UNSW_Rocketry_Senior_Flight_Computer"
 				(path "/9e0253f5-fba5-4205-8256-7fc47a91dd1e/57914cc3-efa9-43f1-a4d3-11a42d51adab"
-					(reference "#PWR093")
+					(reference "#PWR087")
 					(unit 1)
 				)
@@
 		(in_pos_files yes)
 		(dnp no)
-		(property "Reference" "R39"
+		(property "Reference" "R37"
 			(at 103.378 133.35 0)
 			(show_name no)
@@
 			(project "UNSW_Rocketry_Senior_Flight_Computer"
 				(path "/9e0253f5-fba5-4205-8256-7fc47a91dd1e/57914cc3-efa9-43f1-a4d3-11a42d51adab"
-					(reference "R39")
+					(reference "R37")
 					(unit 1)
 				)
@@
 		(in_pos_files yes)
 		(dnp no)
-		(property "Reference" "R36"
+		(property "Reference" "R35"
 			(at 102.87 95.758 0)
 			(show_name no)
@@
 			(project "UNSW_Rocketry_Senior_Flight_Computer"
 				(path "/9e0253f5-fba5-4205-8256-7fc47a91dd1e/57914cc3-efa9-43f1-a4d3-11a42d51adab"
-					(reference "R36")
+					(reference "R35")
 					(unit 1)
 				)
@@
 		(dnp no)
 		(fields_autoplaced yes)
-		(property "Reference" "D15"
+		(property "Reference" "D16"
 			(at 119.6975 67.31 0)
 			(show_name no)
@@
 			)
 		)
-		(property "Value" "LED"
+		(property "Value" "LED_GREEN"
 			(at 119.6975 69.85 0)
 			(show_name no)
@@
 			(project "UNSW_Rocketry_Senior_Flight_Computer"
 				(path "/9e0253f5-fba5-4205-8256-7fc47a91dd1e/57914cc3-efa9-43f1-a4d3-11a42d51adab"
-					(reference "D15")
+					(reference "D16")
 					(unit 1)
 				)
@@
 		(dnp no)
 		(fields_autoplaced yes)
-		(property "Reference" "#PWR092"
+		(property "Reference" "#PWR093"
 			(at 128.27 135.89 0)
 			(hide yes)
@@
 			(project "UNSW_Rocketry_Senior_Flight_Computer"
 				(path "/9e0253f5-fba5-4205-8256-7fc47a91dd1e/57914cc3-efa9-43f1-a4d3-11a42d51adab"
-					(reference "#PWR092")
+					(reference "#PWR093")
 					(unit 1)
 				)
@@
 		(in_pos_files yes)
 		(dnp no)
-		(property "Reference" "R38"
+		(property "Reference" "R33"
 			(at 99.06 124.968 0)
 			(show_name no)
@@
 			(project "UNSW_Rocketry_Senior_Flight_Computer"
 				(path "/9e0253f5-fba5-4205-8256-7fc47a91dd1e/57914cc3-efa9-43f1-a4d3-11a42d51adab"
-					(reference "R38")
+					(reference "R33")
 					(unit 1)
 				)
@@
 		(in_pos_files yes)
 		(dnp no)
-		(property "Reference" "R37"
+		(property "Reference" "R34"
 			(at 102.87 90.678 0)
 			(show_name no)
@@
 			(project "UNSW_Rocketry_Senior_Flight_Computer"
 				(path "/9e0253f5-fba5-4205-8256-7fc47a91dd1e/57914cc3-efa9-43f1-a4d3-11a42d51adab"
-					(reference "R37")
+					(reference "R34")
 					(unit 1)
 				)
@@
 		(dnp no)
 		(fields_autoplaced yes)
-		(property "Reference" "D14"
+		(property "Reference" "D15"
 			(at 119.6975 48.26 0)
 			(show_name no)
@@
 			)
 		)
-		(property "Value" "LED"
+		(property "Value" "LED_RED"
 			(at 119.6975 50.8 0)
 			(show_name no)
@@
 			(project "UNSW_Rocketry_Senior_Flight_Computer"
 				(path "/9e0253f5-fba5-4205-8256-7fc47a91dd1e/57914cc3-efa9-43f1-a4d3-11a42d51adab"
-					(reference "D14")
+					(reference "D15")
 					(unit 1)
 				)
@@
 		(in_pos_files yes)
 		(dnp no)
-		(property "Reference" "R35"
+		(property "Reference" "R36"
 			(at 102.87 100.838 0)
 			(show_name no)
@@
 			(project "UNSW_Rocketry_Senior_Flight_Computer"
 				(path "/9e0253f5-fba5-4205-8256-7fc47a91dd1e/57914cc3-efa9-43f1-a4d3-11a42d51adab"
-					(reference "R35")
+					(reference "R36")
 					(unit 1)
 				)
@@
 		(dnp no)
 		(fields_autoplaced yes)
-		(property "Reference" "#PWR089"
+		(property "Reference" "#PWR088"
 			(at 132.08 93.98 0)
 			(hide yes)
@@
 			(project "UNSW_Rocketry_Senior_Flight_Computer"
 				(path "/9e0253f5-fba5-4205-8256-7fc47a91dd1e/57914cc3-efa9-43f1-a4d3-11a42d51adab"
-					(reference "#PWR089")
+					(reference "#PWR088")
 					(unit 1)
 				)
@@
 		(dnp no)
 		(fields_autoplaced yes)
-		(property "Reference" "R33"
+		(property "Reference" "R38"
 			(at 109.22 49.53 0)
 			(show_name no)
@@
 			(project "UNSW_Rocketry_Senior_Flight_Computer"
 				(path "/9e0253f5-fba5-4205-8256-7fc47a91dd1e/57914cc3-efa9-43f1-a4d3-11a42d51adab"
-					(reference "R33")
+					(reference "R38")
 					(unit 1)
 				)
@@
 			)
 		)
-		(property "Footprint" "Buzzer_Beeper:Buzzer_CUI_CMT-8504-SMT-TR"
+		(property "Footprint" "Buzzer_Beeper:Buzzer_CUI_CPT-9019S-SMT"
 			(at 128.27 133.985 90)
 			(hide yes)
@@
 		(dnp no)
 		(fields_autoplaced yes)
-		(property "Reference" "D16"
+		(property "Reference" "D14"
 			(at 115.57 86.36 0)
 			(show_name no)
@@
 			(project "UNSW_Rocketry_Senior_Flight_Computer"
 				(path "/9e0253f5-fba5-4205-8256-7fc47a91dd1e/57914cc3-efa9-43f1-a4d3-11a42d51adab"
-					(reference "D16")
-					(unit 1)
-				)
+					(reference "D14")
+					(unit 1)
+				)
