File: Comms.kicad_sch (KiCad schematic)
At the start: 1 part, among them J4 USB_C_Receptacle_USB2.0_16P

Commit message: feat: Comms complete
Parts:
- added C23: 1.0uF, PCM_SparkFun-Capacitor:C_0603_1608Metric, symbol PCM_SparkFun-Capacitor:1.0uF_0603_16V_10%
- added C25: 0.1uF, PCM_SparkFun-Capacitor:C_0603_1608Metric, symbol PCM_SparkFun-Capacitor:0.1uF_0603_25V_20%
- added D1: B5819W, Diode_SMD:D_SOD-123, symbol Device:D_Schottky_Small
- added J5: Conn_01x04, Connector_PinHeader_2.54mm:PinHeader_1x04_P2.54mm_Vertical, symbol Connector_Generic:Conn_01x04
- added J6: SWD, Connector_PinHeader_2.54mm:PinHeader_1x05_P2.54mm_Vertical, symbol Connector:Conn_01x05_Pin
- added R2, R3: 5.1k, PCM_SparkFun-Resistor:R_0603_1608Metric, symbol PCM_SparkFun-Resistor:5.1k_0603
- added U6: USBLC6-2SC6, Package_TO_SOT_SMD:SOT-23-6, symbol Power_Protection:USBLC6-2SC6
Connections:
- net GND: now reaches J4.A1 (GND), J4.A12 (GND), J4.B1 (GND), J4.B12 (GND)
- net GND: now also J4.SH (SHIELD), C23.1, C25.1, J5.1 (Pin_1), J6.4 (Pin_4), R2.2, R3.2, U6.2 (GND)
- net at J4.A4 (VBUS), J4.A9 (VBUS), J4.B4 (VBUS)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: now also C23.2, C25.2, D1.2 (A), U6.5 (VBUS)
- net at J4.A5 (CC1): now also R2.1
- net at J4.A6 (D+): now also J4.B6 (D+), U6.6 (I/O1)
- net at J4.A7 (D-): now also J4.B7 (D-), U6.4 (I/O2)
- net at J4.B5 (CC2): now also R3.1
- new net +3.3V: J5.4 (Pin_4), J6.1 (Pin_1)
- new net NRST: J6.5 (Pin_5)
- new net SWCLK: J6.3 (Pin_3)
- new net SWDIO: J6.2 (Pin_2)
- new net UART_RX: J5.3 (Pin_3)
- new net UART_TX: J5.2 (Pin_2)
- new net USB_N: U6.3 (I/O2)
- new net USB_P: U6.1 (I/O1)
- new net VBAT_FUSED: D1.1 (K)
- no-connect marks 0 -> 2
Other:
- moved on the sheet: J4

Commit message: feat: finish schematic (Full)
Parts:
- J3: renamed from J4; footprint (none) -> Connector_USB:USB_C_Receptacle_GCT_USB4085
- renumbered C23 to C29, C25 to C30, D1 to D8, J6 to J4, R2 to R13, R3 to R14, U6 to U8
Changed lines of the file:
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@@
 		(dnp no)
 		(fields_autoplaced yes)
-		(property "Reference" "#PWR056"
+		(property "Reference" "#PWR060"
 			(at 43.18 107.95 0)
 			(hide yes)
@@
 			(project "UNSW_Rocketry_Senior_Flight_Computer"
 				(path "/9e0253f5-fba5-4205-8256-7fc47a91dd1e/4243282c-f3ca-4105-833d-42ac8b978054"
-					(reference "#PWR056")
+					(reference "#PWR060")
 					(unit 1)
 				)
@@
 		(in_pos_files yes)
 		(dnp no)
-		(property "Reference" "C25"
+		(property "Reference" "C30"
 			(at 74.93 53.594 90)
 			(show_name no)
@@
 			(project "UNSW_Rocketry_Senior_Flight_Computer"
 				(path "/9e0253f5-fba5-4205-8256-7fc47a91dd1e/4243282c-f3ca-4105-833d-42ac8b978054"
-					(reference "C25")
+					(reference "C30")
 					(unit 1)
 				)
@@
 		(dnp no)
 		(fields_autoplaced yes)
-		(property "Reference" "#PWR060"
+		(property "Reference" "#PWR062"
 			(at 82.55 63.5 0)
 			(hide yes)
@@
 			(project "UNSW_Rocketry_Senior_Flight_Computer"
 				(path "/9e0253f5-fba5-4205-8256-7fc47a91dd1e/4243282c-f3ca-4105-833d-42ac8b978054"
-					(reference "#PWR060")
+					(reference "#PWR062")
 					(unit 1)
 				)
@@
 		(dnp no)
 		(fields_autoplaced yes)
-		(property "Reference" "D1"
+		(property "Reference" "D8"
 			(at 73.66 36.5759 90)
 			(show_name no)
@@
 			(project "UNSW_Rocketry_Senior_Flight_Computer"
 				(path "/9e0253f5-fba5-4205-8256-7fc47a91dd1e/4243282c-f3ca-4105-833d-42ac8b978054"
-					(reference "D1")
+					(reference "D8")
 					(unit 1)
 				)
@@
 		(dnp no)
 		(fields_autoplaced yes)
-		(property "Reference" "#PWR061"
+		(property "Reference" "#PWR063"
 			(at 91.44 46.99 0)
 			(hide yes)
@@
 			(project "UNSW_Rocketry_Senior_Flight_Computer"
 				(path "/9e0253f5-fba5-4205-8256-7fc47a91dd1e/4243282c-f3ca-4105-833d-42ac8b978054"
-					(reference "#PWR061")
+					(reference "#PWR063")
 					(unit 1)
 				)
@@
 		(dnp no)
 		(fields_autoplaced yes)
-		(property "Reference" "#PWR069"
+		(property "Reference" "#PWR068"
 			(at 175.26 55.88 0)
 			(hide yes)
@@
 			(project "UNSW_Rocketry_Senior_Flight_Computer"
 				(path "/9e0253f5-fba5-4205-8256-7fc47a91dd1e/4243282c-f3ca-4105-833d-42ac8b978054"
-					(reference "#PWR069")
+					(reference "#PWR068")
 					(unit 1)
 				)
@@
 		(in_pos_files yes)
 		(dnp no)
-		(property "Reference" "U6"
+		(property "Reference" "U8"
 			(at 84.7089 81.28 0)
 			(show_name no)
@@
 			(project "UNSW_Rocketry_Senior_Flight_Computer"
 				(path "/9e0253f5-fba5-4205-8256-7fc47a91dd1e/4243282c-f3ca-4105-833d-42ac8b978054"
-					(reference "U6")
+					(reference "U8")
 					(unit 1)
 				)
@@
 		(in_pos_files yes)
 		(dnp no)
-		(property "Reference" "C23"
+		(property "Reference" "C29"
 			(at 80.264 41.402 90)
 			(show_name no)
@@
 			(project "UNSW_Rocketry_Senior_Flight_Computer"
 				(path "/9e0253f5-fba5-4205-8256-7fc47a91dd1e/4243282c-f3ca-4105-833d-42ac8b978054"
-					(reference "C23")
+					(reference "C29")
 					(unit 1)
 				)
@@
 		(dnp no)
 		(fields_autoplaced yes)
-		(property "Reference" "J6"
+		(property "Reference" "J4"
 			(at 139.7 127 90)
 			(show_name no)
@@
 			(project "UNSW_Rocketry_Senior_Flight_Computer"
 				(path "/9e0253f5-fba5-4205-8256-7fc47a91dd1e/4243282c-f3ca-4105-833d-42ac8b978054"
-					(reference "J6")
+					(reference "J4")
 					(unit 1)
 				)
@@
 		(in_pos_files yes)
 		(dnp no)
-		(property "Reference" "R2"
+		(property "Reference" "R13"
 			(at 68.58 57.658 0)
 			(show_name no)
@@
 			(project "UNSW_Rocketry_Senior_Flight_Computer"
 				(path "/9e0253f5-fba5-4205-8256-7fc47a91dd1e/4243282c-f3ca-4105-833d-42ac8b978054"
-					(reference "R2")
+					(reference "R13")
 					(unit 1)
 				)
@@
 		(dnp no)
 		(fields_autoplaced yes)
-		(property "Reference" "#PWR070"
+		(property "Reference" "#PWR069"
 			(at 175.26 72.39 0)
 			(hide yes)
@@
 			(project "UNSW_Rocketry_Senior_Flight_Computer"
 				(path "/9e0253f5-fba5-4205-8256-7fc47a91dd1e/4243282c-f3ca-4105-833d-42ac8b978054"
-					(reference "#PWR070")
+					(reference "#PWR069")
 					(unit 1)
 				)
@@
 		(dnp no)
 		(fields_autoplaced yes)
-		(property "Reference" "#PWR059"
+		(property "Reference" "#PWR061"
 			(at 82.55 60.96 0)
 			(hide yes)
@@
 			(project "UNSW_Rocketry_Senior_Flight_Computer"
 				(path "/9e0253f5-fba5-4205-8256-7fc47a91dd1e/4243282c-f3ca-4105-833d-42ac8b978054"
-					(reference "#PWR059")
+					(reference "#PWR061")
 					(unit 1)
 				)
@@
 		(in_pos_files yes)
 		(dnp no)
-		(property "Reference" "R3"
+		(property "Reference" "R14"
 			(at 68.58 65.532 0)
 			(show_name no)
@@
 			(project "UNSW_Rocketry_Senior_Flight_Computer"
 				(path "/9e0253f5-fba5-4205-8256-7fc47a91dd1e/4243282c-f3ca-4105-833d-42ac8b978054"
-					(reference "R3")
+					(reference "R14")
 					(unit 1)
 				)
@@
 		(in_pos_files yes)
 		(dnp no)
-		(property "Reference" "#PWR067"
+		(property "Reference" "#PWR066"
 			(at 128.27 146.05 0)
 			(hide yes)
@@
 			(project "UNSW_Rocketry_Senior_Flight_Computer"
 				(path "/9e0253f5-fba5-4205-8256-7fc47a91dd1e/4243282c-f3ca-4105-833d-42ac8b978054"
-					(reference "#PWR067")
+					(reference "#PWR066")
 					(unit 1)
 				)
@@
 		(dnp no)
 		(fields_autoplaced yes)
-		(property "Reference" "J4"
+		(property "Reference" "J3"
 			(at 46.99 48.26 0)
 			(show_name no)
@@
 			)
 		)
-		(property "Footprint" ""
+		(property "Footprint" "Connector_USB:USB_C_Receptacle_GCT_USB4085"
 			(at 50.8 71.12 0)
 			(hide yes)
@@
 			(project "UNSW_Rocketry_Senior_Flight_Computer"
 				(path "/9e0253f5-fba5-4205-8256-7fc47a91dd1e/4243282c-f3ca-4105-833d-42ac8b978054"
-					(reference "J4")
+					(reference "J3")
 					(unit 1)
 				)
@@
 		(dnp no)
 		(fields_autoplaced yes)
-		(property "Reference" "#PWR068"
+		(property "Reference" "#PWR067"
 			(at 143.51 142.24 0)
 			(hide yes)
@@
 			(project "UNSW_Rocketry_Senior_Flight_Computer"
 				(path "/9e0253f5-fba5-4205-8256-7fc47a91dd1e/4243282c-f3ca-4105-833d-42ac8b978054"
-					(reference "#PWR068")
+					(reference "#PWR067")
 					(unit 1)
 				)
@@
 		(dnp no)
 		(fields_autoplaced yes)
-		(property "Reference" "#PWR062"
+		(property "Reference" "#PWR064"
 			(at 91.44 50.8 0)
 			(hide yes)
@@
 			(project "UNSW_Rocketry_Senior_Flight_Computer"
 				(path "/9e0253f5-fba5-4205-8256-7fc47a91dd1e/4243282c-f3ca-4105-833d-42ac8b978054"
-					(reference "#PWR062")
+					(reference "#PWR064")
 					(unit 1)
 				)
@@
 		(dnp no)
 		(fields_autoplaced yes)
-		(property "Reference" "#PWR066"
+		(property "Reference" "#PWR065"
 			(at 86.36 58.42 0)
 			(hide yes)
@@
 			(project "UNSW_Rocketry_Senior_Flight_Computer"
 				(path "/9e0253f5-fba5-4205-8256-7fc47a91dd1e/4243282c-f3ca-4105-833d-42ac8b978054"
-					(reference "#PWR066")
-					(unit 1)
-				)
+					(reference "#PWR065")
+					(unit 1)
+				)

Commit message: feat: PCB Designed (Silk screen adjustments)
Connections:
- net USB_RAW_N: now reaches J3.A7 (D-), J3.B7 (D-), U8.4 (I/O2)
- net USB_RAW_P: now reaches J3.A6 (D+), J3.B6 (D+), U8.6 (I/O1)
Changed lines of the file:
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@@
+		)
+	)
+	(label "USB_RAW_N"
+		(at 68.58 71.12 0)
+		(effects
+			(font
+				(size 1.27 1.27)
+			)
+			(justify left bottom)
+		)
+	)
+	(label "USB_RAW_P"
+		(at 68.58 73.66 0)
+		(effects
+			(font
+				(size 1.27 1.27)
+			)
+			(justify left bottom)
 		)
 	)
