File: v1.0/UNSW_Rocketry_Senior_Flight_Computer.kicad_pcb (KiCad board)
At the start: 4 copper layers, 80 x 50 mm, 129 parts, among them J1 SWD, J10 J_BATT, J2 Micro_SD_Card_Det1, J3 USB_C_Receptacle_USB2.0_16P, J5 Conn_01x04, J7 J_PYRO1, J8 J_PYRO2, J9 J_PYRO_BAT, Q1 DMG2301L, Q2 AO3401A, Q3 AO3400A, Q4 AO3400A, Q5 AO3400A, U1 STM32L452RETx, U10 PC817, U11 PC817, U2 TPS63060, U3 SPX3819M5-L-3-3, U4 H3LIS331DL, U5 MS5611 #1, U6 LIS3DH, U7 MS5611 #2, U8 USBLC6-2SC6, U9 PC817, Y1 8MHz

Commit message: fixes
Routing:
- net GND: track 168.4 -> 181.9 mm, vias 36 -> 39
- net PYRO_GND: track 48.1 -> 45.8 mm
- net CS_MS5611_1: track 22.7 -> 24.2 mm
- net +3.3V: track 73.4 -> 74.8 mm, vias 12 -> 13
Changed lines of the file:
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@@
 	)
 	(segment
+		(start 135.983003 92.825)
+		(end 135.658003 92.5)
+		(width 0.25)
+		(layer "F.Cu")
+		(net "+3.3V")
+	)
+	(segment
 		(start 152 90.225)
 		(end 152 91.75)
@@
 	)
 	(segment
+		(start 136.95 92.825)
+		(end 135.983003 92.825)
+		(width 0.25)
+		(layer "F.Cu")
+		(net "+3.3V")
+	)
+	(segment
 		(start 173.6375 100.37)
 		(end 175.0875 100.37)
@@
 	)
 	(via
+		(at 135.658003 92.5)
+		(size 0.6)
+		(drill 0.3)
+		(layers "F.Cu" "B.Cu")
+		(net "+3.3V")
+	)
+	(via
 		(at 151.614827 98.855363)
 		(size 0.6)
@@
 	)
 	(segment
+		(start 158.2117 78.571)
+		(end 159 78.571)
+		(width 0.6)
+		(layer "F.Cu")
+		(net "GND")
+	)
+	(segment
+		(start 141.3 79.9)
+		(end 141.5 79.7)
+		(width 0.25)
+		(layer "F.Cu")
+		(net "GND")
+	)
+	(segment
 		(start 135.35 79.735)
 		(end 135.35 80.65)
@@
 	)
 	(segment
+		(start 141.1 86.525)
+		(end 141.1 86.31005)
+		(width 0.25)
+		(layer "F.Cu")
+		(net "GND")
+	)
+	(segment
 		(start 170.7875 114.7)
 		(end 170.8375 114.65)
@@
 	)
 	(segment
+		(start 157.81 80.468)
+		(end 157.81 78.9727)
+		(width 0.6)
+		(layer "F.Cu")
+		(net "GND")
+	)
+	(segment
 		(start 176.1875 115.06)
 		(end 178.2575 115.06)
@@
 	)
 	(segment
+		(start 160.35 80.468)
+		(end 161.62 80.468)
+		(width 0.6)
+		(layer "F.Cu")
+		(net "GND")
+	)
+	(segment
 		(start 153.525 90.25)
 		(end 153.55 90.225)
@@
 	)
 	(segment
+		(start 180.225 92.3775)
+		(end 180.2525 92.35)
+		(width 1)
+		(layer "F.Cu")
+		(net "GND")
+	)
+	(segment
 		(start 168.2 114.15)
 		(end 168.2 113.45)
@@
 	)
 	(segment
+		(start 159 78.571)
+		(end 159.7483 78.571)
+		(width 0.6)
+		(layer "F.Cu")
+		(net "GND")
+	)
+	(segment
 		(start 142.75 89.9)
 		(end 142.75 90.835786)
@@
 	)
 	(segment
+		(start 157.81 78.9727)
+		(end 158.2117 78.571)
+		(width 0.6)
+		(layer "F.Cu")
+		(net "GND")
+	)
+	(segment
 		(start 138.45 102.075)
 		(end 139.475 102.075)
@@
 	)
 	(segment
+		(start 141.2975 80.435)
+		(end 141.2975 79.9)
+		(width 0.25)
+		(layer "F.Cu")
+		(net "GND")
+	)
+	(segment
+		(start 159 78.571)
+		(end 159 78)
+		(width 0.6)
+		(layer "F.Cu")
+		(net "GND")
+	)
+	(segment
+		(start 141.2975 79.9)
+		(end 141.3 79.9)
+		(width 0.25)
+		(layer "F.Cu")
+		(net "GND")
+	)
+	(segment
 		(start 136.4 87.95)
 		(end 135.4 87.95)
@@
 	)
 	(segment
+		(start 180.225 93.9)
+		(end 180.225 92.3775)
+		(width 1)
+		(layer "F.Cu")
+		(net "GND")
+	)
+	(segment
 		(start 152.825 80.4975)
 		(end 153.325 80.4975)
@@
 	)
 	(segment
+		(start 160.35 79.1727)
+		(end 160.35 80.468)
+		(width 0.6)
+		(layer "F.Cu")
+		(net "GND")
+	)
+	(segment
 		(start 152.35 79.647068)
 		(end 153.224568 78.7725)
@@
 	)
 	(segment
+		(start 141.1 86.31005)
+		(end 140.5 85.71005)
+		(width 0.25)
+		(layer "F.Cu")
+		(net "GND")
+	)
+	(segment
 		(start 178.2575 115.06)
 		(end 178.2575 115.8575)
@@
 	)
 	(segment
+		(start 142.1 79.7)
+		(end 142.2975 79.8975)
+		(width 0.25)
+		(layer "F.Cu")
+		(net "GND")
+	)
+	(segment
 		(start 152.074568 79.9225)
 		(end 152.35 79.9225)
@@
 	)
 	(segment
+		(start 153.325 80.4975)
+		(end 153.325 81.025)
+		(width 0.2)
+		(layer "F.Cu")
+		(net "GND")
+	)
+	(segment
 		(start 138 92.325)
 		(end 136.95 91.275)
@@
 	)
 	(segment
+		(start 159.7483 78.571)
+		(end 160.35 79.1727)
+		(width 0.6)
+		(layer "F.Cu")
+		(net "GND")
+	)
+	(segment
 		(start 152.125 99.475)
 		(end 152.15 99.45)
@@
 	)
 	(segment
+		(start 153.325 81.025)
+		(end 153.7 81.4)
+		(width 0.2)
+		(layer "F.Cu")
+		(net "GND")
+	)
+	(segment
 		(start 136.35 111.1)
 		(end 136.35 118.95)
@@
 	)
 	(segment
+		(start 142.2975 79.8975)
+		(end 142.2975 80.435)
+		(width 0.25)
+		(layer "F.Cu")
+		(net "GND")
+	)
+	(segment
 		(start 162.5 109.3)
 		(end 162.5 107.6)
@@
 		(net "GND")
 	)
+	(segment
+		(start 141.5 79.7)
+		(end 142.1 79.7)
+		(width 0.25)
+		(layer "F.Cu")
+		(net "GND")
+	)
 	(via
 		(at 150.574265 77.5)
@@
 	)
 	(via
+		(at 159 78)
+		(size 0.6)
+		(drill 0.3)
+		(layers "F.Cu" "B.Cu")
+		(net "GND")
+	)
+	(via
 		(at 139.7 102.3)
 		(size 0.6)
@@
 	)
 	(via
+		(at 153.7 81.4)
+		(size 0.6)
+		(drill 0.3)
+		(layers "F.Cu" "B.Cu")
+		(net "GND")
+	)
+	(via
 		(at 135.35 87.9)
 		(size 0.6)
@@
 	)
 	(via
+		(at 140.5 85.71005)
+		(size 0.6)
+		(drill 0.3)
+		(layers "F.Cu" "B.Cu")
+		(net "GND")
+	)
+	(via
 		(at 154.75 90.2)
 		(size 0.6)
@@
 	)
 	(segment
+		(start 147.389602 82.1475)
+		(end 146.35 83.187102)
+		(width 0.5)
+		(layer "F.Cu")
+		(net "CS_MS5611_1")
+	)
+	(segment
 		(start 142.605588 97.325)
 		(end 143.23792 96.692668)
@@
 	(segment
 		(start 147.4975 82.1475)
+		(end 147.389602 82.1475)
+		(width 0.5)
+		(layer "F.Cu")
+		(net "CS_MS5611_1")
+	)
+	(segment
+		(start 147.4975 82.1475)
 		(end 149.6475 82.1475)
 		(width 0.5)
@@
 	)
 	(segment
-		(start 133.55 89.4)
-		(end 134.75 90.6)
-		(width 0.75)
-		(layer "F.Cu")
-		(net "PYRO_GND")
-	)
-	(segment
 		(start 125.85 92.85)
 		(end 125.85 93.2)
@@
 	)
 	(segment
+		(start 133 89.4)
+		(end 127.2 89.4)
+		(width 0.75)
+		(layer "F.Cu")
+		(net "PYRO_GND")
+	)
+	(segment
 		(start 133 107.35)
 		(end 127.5 107.35)
@@
 	)
 	(segment
-		(start 127.2 89.4)
-		(end 133.55 89.4)
-		(width 0.75)
-		(layer "F.Cu")
-		(net "PYRO_GND")
-	)
-	(segment
 		(start 132.35 102.375)
 		(end 133.575 102.375)
@@
 	)
 	(via
-		(at 134.75 90.6)
+		(at 133 89.4)
 		(size 1)
 		(drill 0.5)

Commit message: Fix: Tims review changes
Connections:
- H1 pad 1: (no net) -> GND
- H2 pad 1: (no net) -> GND
- H3 pad 1: (no net) -> GND
- H4 pad 1: (no net) -> GND
Routing:
- net SDMMC_D0: track 6.31 -> 9.69 mm, vias 0 -> 2
- net /Comms/USB_RAW_P: track 5.34 -> 6.18 mm, vias 0 -> 1
- net /Comms/USB_RAW_N: track 7.65 -> 7.61 mm, vias 1 -> 0
Changed lines of the file:
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@@
 			(layers "*.Cu" "*.Mask")
 			(remove_unused_layers no)
+			(net "GND")
 			(zone_connect 2)
 		)
@@
 			(layers "*.Cu" "*.Mask")
 			(remove_unused_layers no)
+			(net "GND")
 			(zone_connect 2)
 		)
@@
 			(layers "*.Cu" "*.Mask")
 			(remove_unused_layers no)
+			(net "GND")
 			(zone_connect 2)
 		)
@@
 			(layers "*.Cu" "*.Mask")
 			(remove_unused_layers no)
+			(net "GND")
 			(zone_connect 2)
 		)
@@
 	)
 	(segment
-		(start 158.025 118.335661)
-		(end 158.875 119.185661)
+		(start 157.321717 115.746717)
+		(end 157.877571 115.746717)
 		(width 0.4)
 		(layer "F.Cu")
@@
 	)
 	(segment
-		(start 158.025 116.150001)
-		(end 158.025 118.125)
+		(start 156.7625 115.1875)
+		(end 157.321717 115.746717)
 		(width 0.4)
 		(layer "F.Cu")
 		(net "/Comms/USB_RAW_P")
 	)
+	(via
+		(at 157.877571 115.746717)
+		(size 0.6)
+		(drill 0.3)
+		(layers "F.Cu" "B.Cu")
+		(net "/Comms/USB_RAW_P")
+	)
 	(segment
 		(start 158.025 118.125)
-		(end 158.025 118.335661)
+		(end 158.025 117.575)
 		(width 0.4)
-		(layer "F.Cu")
+		(layer "B.Cu")
 		(net "/Comms/USB_RAW_P")
 	)
 	(segment
-		(start 158.875 119.185661)
-		(end 158.875 119.475)
+		(start 158.246717 115.746717)
+		(end 158.6 116.1)
 		(width 0.4)
-		(layer "F.Cu")
+		(layer "B.Cu")
 		(net "/Comms/USB_RAW_P")
 	)
 	(segment
-		(start 156.7625 115.1875)
-		(end 157.062499 115.1875)
+		(start 158.875 119.475)
+		(end 158.875 119.264339)
 		(width 0.4)
-		(layer "F.Cu")
+		(layer "B.Cu")
 		(net "/Comms/USB_RAW_P")
 	)
 	(segment
-		(start 157.062499 115.1875)
-		(end 158.025 116.150001)
+		(start 158.025 118.414339)
+		(end 158.025 118.125)
 		(width 0.4)
-		(layer "F.Cu")
+		(layer "B.Cu")
 		(net "/Comms/USB_RAW_P")
 	)
 	(segment
-		(start 157.247182 116.65)
-		(end 157.3 116.597182)
+		(start 158.025 117.575)
+		(end 158.6 117)
 		(width 0.4)
-		(layer "F.Cu")
-		(net "/Comms/USB_RAW_N")
+		(layer "B.Cu")
+		(net "/Comms/USB_RAW_P")
 	)
 	(segment
-		(start 154.8625 115.1875)
-		(end 154.8625 115.849999)
+		(start 158.875 119.264339)
+		(end 158.025 118.414339)
 		(width 0.4)
-		(layer "F.Cu")
-		(net "/Comms/USB_RAW_N")
+		(layer "B.Cu")
+		(net "/Comms/USB_RAW_P")
 	)
 	(segment
-		(start 154.8625 115.849999)
-		(end 155.662501 116.65)
+		(start 157.877571 115.746717)
+		(end 158.246717 115.746717)
 		(width 0.4)
-		(layer "F.Cu")
-		(net "/Comms/USB_RAW_N")
+		(layer "B.Cu")
+		(net "/Comms/USB_RAW_P")
 	)
 	(segment
-		(start 155.662501 116.65)
-		(end 157.247182 116.65)
+		(start 158.6 117)
+		(end 158.6 116.1)
+		(width 0.4)
+		(layer "B.Cu")
+		(net "/Comms/USB_RAW_P")
+	)
+	(segment
+		(start 158.025 119.475)
+		(end 158.025 119.185661)
 		(width 0.4)
 		(layer "F.Cu")
 		(net "/Comms/USB_RAW_N")
 	)
-	(via
-		(at 157.3 116.597182)
-		(size 0.6)
-		(drill 0.3)
-		(layers "F.Cu" "B.Cu")
+	(segment
+		(start 158.875 118.125)
+		(end 158.875 117.630026)
+		(width 0.4)
+		(layer "F.Cu")
 		(net "/Comms/USB_RAW_N")
 	)
 	(segment
-		(start 158.875 118.414339)
-		(end 158.025 119.264339)
+		(start 158.025 119.185661)
+		(end 158.875 118.335661)
 		(width 0.4)
-		(layer "B.Cu")
+		(layer "F.Cu")
 		(net "/Comms/USB_RAW_N")
 	)
 	(segment
-		(start 157.842156 116.597182)
-		(end 157.3 116.597182)
+		(start 158.875 117.630026)
+		(end 157.894974 116.65)
 		(width 0.4)
-		(layer "B.Cu")
+		(layer "F.Cu")
 		(net "/Comms/USB_RAW_N")
 	)
 	(segment
-		(start 158.875 118.125)
-		(end 158.875 117.630026)
+		(start 158.875 118.335661)
+		(end 158.875 118.125)
 		(width 0.4)
-		(layer "B.Cu")
+		(layer "F.Cu")
 		(net "/Comms/USB_RAW_N")
 	)
 	(segment
-		(start 158.025 119.264339)
-		(end 158.025 119.475)
+		(start 155.662501 116.65)
+		(end 154.8625 115.849999)
 		(width 0.4)
-		(layer "B.Cu")
+		(layer "F.Cu")
 		(net "/Comms/USB_RAW_N")
 	)
 	(segment
-		(start 158.875 118.125)
-		(end 158.875 118.414339)
+		(start 157.894974 116.65)
+		(end 155.662501 116.65)
 		(width 0.4)
-		(layer "B.Cu")
+		(layer "F.Cu")
 		(net "/Comms/USB_RAW_N")
 	)
 	(segment
-		(start 158.875 117.630026)
-		(end 157.842156 116.597182)
+		(start 154.8625 115.849999)
+		(end 154.8625 115.1875)
 		(width 0.4)
-		(layer "B.Cu")
+		(layer "F.Cu")
 		(net "/Comms/USB_RAW_N")
 	)
@@
 	)
 	(segment
-		(start 142.789224 102.35)
-		(end 143.65 102.35)
+		(start 141.291942 104.091942)
+		(end 141.291942 103.847282)
 		(width 0.25)
 		(layer "F.Cu")
@@
 	)
 	(segment
-		(start 143.65 102.35)
-		(end 143.75 102.25)
+		(start 142.789224 102.35)
+		(end 143.65 102.35)
 		(width 0.25)
 		(layer "F.Cu")
@@
 	)
 	(segment
-		(start 140.95 104.189224)
+		(start 141.291942 103.847282)
 		(end 142.789224 102.35)
 		(width 0.25)
@@
 	)
 	(segment
-		(start 140.95 105.9)
-		(end 140.95 104.189224)
+		(start 140.9 105.95)
+		(end 140.95 105.9)
+		(width 0.25)
+		(layer "F.Cu")
+		(net "SDMMC_D0")
+	)
+	(segment
+		(start 140.9 107)
+		(end 140.9 105.95)
+		(width 0.25)
+		(layer "F.Cu")
+		(net "SDMMC_D0")
+	)
+	(segment
+		(start 143.65 102.35)
+		(end 143.75 102.25)
 		(width 0.25)
 		(layer "F.Cu")
 		(net "SDMMC_D0")
 	)
+	(via
+		(at 141.291942 104.091942)
+		(size 0.6)
+		(drill 0.3)
+		(layers "F.Cu" "B.Cu")
+		(net "SDMMC_D0")
+	)
+	(via
+		(at 140.9 107)
+		(size 0.6)
+		(drill 0.3)
+		(layers "F.Cu" "B.Cu")
+		(net "SDMMC_D0")
+	)
+	(segment
+		(start 141.5 107.2)
+		(end 141.9 106.8)
+		(width 0.25)
+		(layer "In2.Cu")
+		(net "SDMMC_D0")
+	)
+	(segment
+		(start 141.1 107.2)
+		(end 140.9 107)
+		(width 0.25)
+		(layer "In2.Cu")
+		(net "SDMMC_D0")
+	)
+	(segment
+		(start 141.9 104.7)
+		(end 141.9 106.8)
+		(width 0.25)
+		(layer "In2.Cu")
+		(net "SDMMC_D0")
+	)
+	(segment
+		(start 141.291942 104.091942)
+		(end 141.9 104.7)
+		(width 0.25)
+		(layer "In2.Cu")
+		(net "SDMMC_D0")
+	)
+	(segment
+		(start 141.5 107.2)
+		(end 141.1 107.2)
+		(width 0.25)
+		(layer "In2.Cu")
+		(net "SDMMC_D0")
+	)
